Commit message: camera adjustments

File: rotors_description/urdf/component_snippets.xacro (robot description, xacro)
@@ -706,5 +706,5 @@
         namespace="${namespace}" parent_link="${namespace}/vi_sensor_link"
         camera_suffix="depth" frame_rate="10.0" max_range="10.0">
-        <origin xyz="0.015 0.055 0.0065" rpy="0 0 0" />
+        <origin xyz="0.015 0.0 0.0065" rpy="0 0 0" />
       </xacro:vi_sensor_depth_macro>
     </xacro:if>

Commit message: Fix build errors and xacro files
Techpod won't load in the simulation world, fixed that and build errors.
Removed mavlink_interface from build pool (As it has errors and is not
required)

File: rotors_description/urdf/component_snippets.xacro (robot description, xacro)
@@ -1092,6 +1092,6 @@
       accelerometer_bias_correlation_time="300.0"
       accelerometer_turn_on_bias_sigma="0.1960">
-      <xacro:cube_inertia l="0.02" mass="0.015" />
-      <xacro:insert_block name="origin" />
+      <inertia ixx="0.00001" ixy="0.0" ixz="0.0" iyy="0.00001" iyz="0.0" izz="0.00001" />
+      <origin xyz="0 0 0" rpy="0 0 0" />
     </xacro:imu_plugin_macro>
   </xacro:macro>

File: rotors_description/urdf/techpod_base.xacro (robot description, xacro)
@@ -37,5 +37,7 @@
   -->
   <!-- Mount an ADIS16448 IMU. -->
-  <xacro:default_imu namespace="${namespace}" parent_link="${namespace}/base_link" />
+  <xacro:default_imu namespace="${namespace}" parent_link="${namespace}/base_link" >
+    <origin xyz="0 0 0" rpy="0 0 0" />
+  </xacro:default_imu>
   <!-- Mount a GPS. -->
   <xacro:default_gps namespace="${namespace}" parent_link="${namespace}/base_link" >
