Commit message: Fix launch files for firefly and hummingbird

File: rotors_description/urdf/firefly_base.xacro (robot description, xacro)
@@ -29,5 +29,7 @@
   </xacro:if>
   <!-- Mount an ADIS16448 IMU. -->
-  <xacro:default_imu namespace="${namespace}" parent_link="${namespace}/base_link" />
+  <xacro:default_imu namespace="${namespace}" parent_link="${namespace}/base_link" >
+    <origin xyz="0.0 0.0 0.0" rpy="0 0 0" />
+  </xacro:default_imu>
   <xacro:if value="$(arg enable_ground_truth)">
     <xacro:ground_truth_imu_and_odometry namespace="${namespace}" parent_link="${namespace}/base_link" />

File: rotors_description/urdf/hummingbird_base.xacro (robot description, xacro)
@@ -27,5 +27,7 @@
   </xacro:if>
   <!-- Mount an ADIS16448 IMU. -->
-  <xacro:default_imu namespace="${namespace}" parent_link="${namespace}/base_link" />
+  <xacro:default_imu namespace="${namespace}" parent_link="${namespace}/base_link" >
+    <origin xyz="0.3 -0.01 0.023" rpy="0 0 0" />
+  </xacro:default_imu>
   <xacro:if value="$(arg enable_ground_truth)">
     <xacro:ground_truth_imu_and_odometry namespace="${namespace}" parent_link="${namespace}/base_link" />
